File: KicadJE_Drum_PE78.kicad_pcb (KiCad board)
At the start: 2 copper layers, 183 x 128 mm, 213 parts, among them J101 Snare, J102 LCymbals, J103 SCymbals, J104 Maracas, J105 Bass, J106 LBongo, J107 HBongo, J108 Claves, J201 AudioJack2_SwitchT, J202 AudioJack2_SwitchT, J203 AudioJack2_SwitchT, J204 Power +, J205 Power -, J206 Conn_01x03_Male, J207 Conn_01x03_Male, J208 Conn_01x03_Male, J209 Conn_01x03_Male, J210 Conn_01x02_Male, J301 Tone/Noise, J302 RND, J303 Noise, J304 DRUM_OUT, J401 Tone/Noise, P101 HEADER_2x8_Doepfer, P201 HEADER_2x5_Doepfer, P401 HEADER_2x8_Doepfer, Q101 2N3904, Q102 2N3904, Q103 2N3904, Q104 2N3904, SW201 SW_SPDT, U101 74HC04, U302 TL072

Commit message: Board labels
Other:
- board text added: "Drum78"
- board text added: "Drum78 - Rev A JE - 27/4-2021"
- board text added: "Johansen Engineering Drum78 Rev A 22/04-2021"
- board text removed: "Johansen Engineering Glide Rev A 22/03-2020"
Changed lines of the file:
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@@
   (general
     (thickness 1.6)
-    (drawings 117)
+    (drawings 119)
     (tracks 798)
     (zones 0)
@@
   (page A4)
   (layers
-    (0 F.Cu signal)
-    (31 B.Cu signal)
+    (0 F.Cu signal hide)
+    (31 B.Cu signal hide)
     (32 B.Adhes user)
-    (33 F.Adhes user hide)
+    (33 F.Adhes user)
     (34 B.Paste user)
-    (35 F.Paste user hide)
+    (35 F.Paste user)
     (36 B.SilkS user)
-    (37 F.SilkS user hide)
+    (37 F.SilkS user)
     (38 B.Mask user)
-    (39 F.Mask user hide)
-    (40 Dwgs.User user hide)
+    (39 F.Mask user)
+    (40 Dwgs.User user)
     (41 Cmts.User user)
     (42 Eco1.User user)
@@
     (45 Margin user)
     (46 B.CrtYd user)
-    (47 F.CrtYd user hide)
+    (47 F.CrtYd user)
     (48 B.Fab user)
-    (49 F.Fab user hide)
+    (49 F.Fab user)
   )
   (setup
@@
     )
   )
+  (gr_text "Drum78 - Rev A\nJE - 27/4-2021 " (at 149.8 148.2) (layer B.SilkS)
+    (effects (font (size 1.2 1) (thickness 0.2)) (justify left mirror))
+  )
+  (gr_text "Drum78\n" (at 146.4 66.6 90) (layer F.SilkS)
+    (effects (font (size 4 2) (thickness 0.5)) (justify left))
+  )
   (gr_line (start 141.8 68) (end 143.2 69.8) (layer B.SilkS) (width 0.12))
   (gr_line (start 141.8 82) (end 143.4 81) (layer B.SilkS) (width 0.12))
@@
     (effects (font (size 1 1) (thickness 0.1)) (justify mirror))
   )
-  (gr_text "Johansen Engineering \nGlide Rev A\n22/03-2020" (at 220.5 153.5) (layer B.SilkS)
+  (gr_text "Johansen Engineering \nDrum78 Rev A\n22/04-2021" (at 220.5 153.5) (layer B.SilkS)
     (effects (font (size 1 1) (thickness 0.25)) (justify left mirror))
   )
