File: KicadJE_Drum_PE78 - Base.kicad_pcb (KiCad board)
At the start: 2 copper layers, 183 x 128 mm, 213 parts, among them J101 Snare, J102 LCymbals, J103 SCymbals, J104 Maracas, J105 Bass, J106 LBongo, J107 HBongo, J108 Claves, J201 AudioJack2_SwitchT, J202 AudioJack2_SwitchT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

Commit message: Base
Routing:
- net Net-(J401-Pad2): track 0.00 -> 6.02 mm
- net Net-(J401-Pad1): track 0.00 -> 3.48 mm
- net GND: track 170.1 -> 173.4 mm, vias 22 -> 24
- net /KicadJE_PDU_1/-12: track 5.24 -> 7.78 mm
- net /KicadJE_PDU_1/+12: track 5.28 -> 7.82 mm
