File: KicadJE_Drum_PE78 - Face.kicad_pcb (KiCad board)
At the start: 2 copper layers, 183 x 128 mm, 213 parts, among them J101 Snare, J102 LCymbals, J103 SCymbals, J104 Maracas, J105 Bass, J106 LBongo, J107 HBongo, J108 Claves, J201 AudioJack2_SwitchT, J202 AudioJack2_SwitchT, J203 AudioJack2_SwitchT, J204 Power +, J205 Power -, J206 Conn_01x03_Male, J207 Conn_01x03_Male, J208 Conn_01x03_Male, J209 Conn_01x03_Male, J210 Conn_01x02_Male, J301 Tone/Noise, J302 RND, J303 Noise, J304 DRUM_OUT, J401 Tone/Noise, P101 HEADER_2x8_Doepfer, P201 HEADER_2x5_Doepfer, P401 HEADER_2x8_Doepfer, Q101 2N3904, Q102 2N3904, Q103 2N3904, Q104 2N3904, SW201 SW_SPDT, U101 74HC04, U302 TL072

Commit message: Faceplate + Gerber
Parts:
- removed C101: 330n, AJ:C_0805_AJ
- removed C102, C107, C120, C130, C203, C204: 100n, AJ:C_0805_AJ
- removed C103, C303, C304: 220n, AJ:C_0805_AJ
- removed C104, C113: 150n, AJ:C_0805_AJ
- removed C105, C109, C114, C115: 47n, AJ:C_0805_AJ
- removed C106, C108: 68n, AJ:C_0805_AJ
- removed C110, C116: 15n, AJ:C_0805_AJ
- removed C111, C112, C119, C124, C301, C302: 4n7, AJ:C_0805_AJ
- removed C117: 22n, AJ:C_0805_AJ
- removed C118, C123: 33n, AJ:C_0805_AJ
- removed C121, C125: 10n, AJ:C_0805_AJ
- removed C122, C126: 1n5, AJ:C_0805_AJ
- removed C127, C128, C129, C201, C202, C401, C403: 1u, AJ:C_0805_AJ
- removed D101, D102, D103, D104, D105, D106, D107, D108: 1N4148, Diode_SMD:D_MiniMELF
- removed D109: On LED, AJ:D_0805_AJ
- removed D110, D111, D203, D204, D404, D405: 1N4007, Diode_SMD:D_MiniMELF
- removed D201: On LED +, AJ:D_0805_AJ
- removed D202: On LED -, AJ:D_0805_AJ
- removed D401: +12V, AJ:D_0805_AJ
- removed D402: +5V, AJ:D_0805_AJ
- removed D403: -12v, AJ:D_0805_AJ
- removed the G*** at (95.0, 127.5)
- removed the G*** at (141.8, 117.8)
- removed the G*** at (58.5, 52.2)
- removed the G*** at (87.5, 95.0)
- removed the G*** at (81.0, 52.2)
- removed the H103 at (107.5, 53.0)
- removed the H103 at (96.5, 53.0)
- removed the H103 at (107.5, 147.2)
- removed the H103 at (96.5, 147.2)
- removed J101: Snare, Connector_Audio:Jack_3.5mm_QingPu_WQP-PJ398SM_Vertical_CircularHoles
- removed J102: LCymbals, Connector_Audio:Jack_3.5mm_QingPu_WQP-PJ398SM_Vertical_CircularHoles
- removed J103: SCymbals, Connector_Audio:Jack_3.5mm_QingPu_WQP-PJ398SM_Vertical_CircularHoles
- removed J104: Maracas, Connector_Audio:Jack_3.5mm_QingPu_WQP-PJ398SM_Vertical_CircularHoles
- removed J105: Bass, Connector_Audio:Jack_3.5mm_QingPu_WQP-PJ398SM_Vertical_CircularHoles
- removed J106: LBongo, Connector_Audio:Jack_3.5mm_QingPu_WQP-PJ398SM_Vertical_CircularHoles
- removed J107: HBongo, Connector_Audio:Jack_3.5mm_QingPu_WQP-PJ398SM_Vertical_CircularHoles
- removed J108: Claves, Connector_Audio:Jack_3.5mm_QingPu_WQP-PJ398SM_Vertical_CircularHoles
- removed J201, J202, J203: AudioJack2_SwitchT, Connector_Audio:Jack_3.5mm_Switronic_ST-005-G_horizontal
- removed J204: Power +, Connector_PinHeader_2.54mm:PinHeader_2x02_P2.54mm_Vertical
- removed J205: Power -, Connector_PinHeader_2.54mm:PinHeader_2x02_P2.54mm_Vertical
- removed J206, J207, J208, J209: Conn_01x03_Male, Connector_PinHeader_2.54mm:PinHeader_1x03_P2.54mm_Vertical
- removed J210: Conn_01x02_Male, Connector_PinHeader_2.54mm:PinHeader_1x02_P2.54mm_Vertical
- removed J301: Tone/Noise, Connector_PinHeader_2.54mm:PinHeader_1x03_P2.54mm_Vertical
- removed J302: RND, Connector_Audio:Jack_3.5mm_QingPu_WQP-PJ398SM_Vertical_CircularHoles
- removed J303: Noise, Connector_Audio:Jack_3.5mm_QingPu_WQP-PJ398SM_Vertical_CircularHoles
- removed J304: DRUM_OUT, Connector_Audio:Jack_3.5mm_QingPu_WQP-PJ398SM_Vertical_CircularHoles
- removed J401: Tone/Noise, Connector_PinHeader_2.54mm:PinHeader_1x04_P2.54mm_Vertical_SMD_Pin1Left
- removed L103, L104: 100mH, Inductor_SMD:L_1206_3216Metric
- removed P101, P401: HEADER_2x8_Doepfer, Connector_IDC:IDC-Header_2x08_P2.54mm_Vertical
- removed P201: HEADER_2x5_Doepfer, Connector_IDC:IDC-Header_2x05_P2.54mm_Vertical
- removed Q101, Q102, Q103, Q104: 2N3904, Package_TO_SOT_SMD:SOT-23_Handsoldering
- removed R101, R103, R116, R117, R139, R140, R308, R309, R311, R405: 10k, AJ:R_0805_AJ
- removed R102, R106, R131, R138, R201, R202, R313, R316, R404, R406: 22k, AJ:R_0805_AJ
- removed R104, R105, R132, R133: 12k, AJ:R_0805_AJ
- removed R107, R108, R134, R135: 47k, AJ:R_0805_AJ
- removed R109, R110, R118, R123, R128: 1M, AJ:R_0805_AJ
- removed R111, R112, R136, R137: 27k, AJ:R_0805_AJ
- removed R113, R301, R302, R307: 100k, AJ:R_0805_AJ
- removed R114: 2k2, AJ:R_0805_AJ
- removed R115, R303: 470k, AJ:R_0805_AJ
- removed R119, R121, R141, R143: 150k, AJ:R_0805_AJ
- removed R120, R122, R125, R127, R142, R144, R148, R150: 68k, AJ:R_0805_AJ
- removed R124, R126, R147, R149: 0-470k, AJ:R_0805_AJ
- removed R129, R130: 4k7, AJ:R_0805_AJ
- removed R145, R146, R151, R203, R204, R407, R408, R409: 10R, AJ:R_0805_AJ
- removed R205, R206, R310: OPEN, AJ:R_0805_AJ
- removed R304, R305, R306: 390k, AJ:R_0805_AJ
- removed R312, R401, R402, R403: 0R, AJ:R_0805_AJ
- removed R314: 1k, AJ:R_0805_AJ
- removed R315: 470r, AJ:R_0805_AJ
- removed R323: 470R, AJ:R_0805_AJ
- removed REF** (x4): MountingHole_8.4mm_M8, MountingHole:MountingHole_8.4mm_M8
- removed RV101: R_POT_TRIM, Potentiometer_THT:Potentiometer_Bourns_3296W_Vertical
- removed RV102: 220k, AJ:Potentiometer_China_RK09_Single_Vertical_AJ
- removed RV201: 100k, AJ:Potentiometer_China_RK09_Single_Vertical_AJ
- removed SW201: SW_SPDT, Button_Switch_THT:SW_PUSH_6mm_H8mm
- removed U101: 74HC04, Package_SO:SO-14_5.3x10.2mm_P1.27mm
- removed U302: TL072, AJ:AJ_SO-8_5.3x6.2mm_P1.27mm
Routing:
- net +12Vc: track 226.4 -> 0.00 mm, vias 4 -> 0
- net +5V: track 174.3 -> 0.00 mm, vias 4 -> 0
- net GND: track 170.1 -> 0.00 mm, vias 22 -> 0
- net -12Vc: track 128.2 -> 0.00 mm, vias 1 -> 0
- net Net-(R323-Pad2): track 106.0 -> 0.00 mm
- net LBongoTrig: track 102.2 -> 0.00 mm, vias 4 -> 0
- net Net-(J301-Pad3): track 97.2 -> 0.00 mm, vias 1 -> 0
- net BassTrig: track 93.2 -> 0.00 mm
- net NoiseOut: track 69.8 -> 0.00 mm, vias 7 -> 0
- net HBongoTrig: track 62.8 -> 0.00 mm, vias 6 -> 0
- net Net-(R315-Pad2): track 60.2 -> 0.00 mm, vias 5 -> 0
- net Net-(J210-Pad1): track 53.7 -> 0.00 mm
- net Net-(J210-Pad2): track 50.2 -> 0.00 mm
- net ClavesTrig: track 46.2 -> 0.00 mm, vias 6 -> 0
- net Net-(C111-Pad2): track 32.0 -> 0.00 mm
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- removed copper zone on F.Cu, net (none)
Other:
- board size 183 x 128 mm -> 40 x 128 mm
- board text removed: "BB-Power"
- board text removed: "Drum78"
- board text removed: "Drum78 - Rev A JE - 27/4-2021"
- board text removed: "KicadJE-BB-Power Johansen Engineering 22/4/2021 Rev A"
- board text removed: "KicadJE-PDU1 27/4/2021 Rev A"
- board text removed: "PDU1"

Commit message: Faceplate - not matching base - fix
Parts:
- removed the TP107 at (223.0, 125.0)
- added C101: 330n, AJ:C_0805_AJ, B.Cu at (123.0, 85.5)
- added C102: 100n, AJ:C_0805_AJ, B.Cu at (117.0, 107.0)
- added C103: 220n, AJ:C_0805_AJ, B.Cu at (120.0, 95.0)
- added C104: 150n, AJ:C_0805_AJ, B.Cu at (117.0, 148.0)
- added C105: 47n, AJ:C_0805_AJ, B.Cu at (117.0, 138.5)
- added C106: 68n, AJ:C_0805_AJ, B.Cu at (123.0, 73.5)
- added C107: 100n, AJ:C_0805_AJ, B.Cu at (123.5, 101.5)
- added C108: 68n, AJ:C_0805_AJ, B.Cu at (121.0, 115.0)
- added C109: 47n, AJ:C_0805_AJ, B.Cu at (148.0, 63.5)
- added C110: 15n, AJ:C_0805_AJ, B.Cu at (148.0, 79.5)
- added C111: 4n7, AJ:C_0805_AJ, B.Cu at (128.5, 102.5)
- added C112: 4n7, AJ:C_0805_AJ, B.Cu at (128.5, 100.5)
- added C113: 150n, AJ:C_0805_AJ, B.Cu at (142.0, 63.5)
- added C114: 47n, AJ:C_0805_AJ, B.Cu at (142.0, 79.5)
- added C115: 47n, AJ:C_0805_AJ, B.Cu at (148.0, 67.5)
- added C116: 15n, AJ:C_0805_AJ, B.Cu at (148.0, 83.5)
- added C117: 22n, AJ:C_0805_AJ, B.Cu at (146.0, 116.5)
- added C118: 33n, AJ:C_0805_AJ, B.Cu at (117.0, 128.5)
- added C119: 4n7, AJ:C_0805_AJ, B.Cu at (117.0, 118.5)
- added C120: 100n, AJ:C_0805_AJ, B.Cu at (142.0, 105.0)
- added C121: 10n, AJ:C_0805_AJ, B.Cu at (148.0, 71.5)
- added C122: 1n5, AJ:C_0805_AJ, B.Cu at (131.5, 83.5)
- added C123: 33n, AJ:C_0805_AJ, B.Cu at (142.0, 71.5)
- added C124: 4n7, AJ:C_0805_AJ, B.Cu at (137.5, 83.5)
- added C125: 10n, AJ:C_0805_AJ, B.Cu at (148.0, 75.5)
- added C126: 1n5, AJ:C_0805_AJ, B.Cu at (131.5, 79.5)
- added C127: 1u, AJ:C_0805_AJ, F.Cu at (131.5, 62.5)
- added C128: 1u, AJ:C_0805_AJ, F.Cu at (124.0, 62.5)
- added C129: 1u, AJ:C_0805_AJ, F.Cu at (136.5, 62.5)
- added C130: 100n, AJ:C_0805_AJ, B.Cu at (135.0, 63.5)
- added C201: 1u, AJ:C_0805_AJ, F.Cu at (79.5, 79.0)
- added C202: 1u, AJ:C_0805_AJ, F.Cu at (79.5, 124.0)
- added C203: 100n, AJ:C_0805_AJ, F.Cu at (137.9, 94.0)
- added C204: 100n, AJ:C_0805_AJ, F.Cu at (141.5, 86.0)
- added C301: 4n7, AJ:C_0805_AJ, B.Cu at (128.0, 71.0)
- added C302: 4n7, AJ:C_0805_AJ, B.Cu at (128.0, 67.0)
- added C303: 220n, AJ:C_0805_AJ, F.Cu at (144.0, 83.0)
- added C304: 220n, AJ:C_0805_AJ, B.Cu at (140.5, 125.0)
- added C401: 1u, AJ:C_0805_AJ, B.Cu at (97.0, 127.0)
- added C403: 1u, AJ:C_0805_AJ, B.Cu at (97.0, 137.2)
- added D101: 1N4148, Diode_SMD:D_MiniMELF, B.Cu at (117.8, 109.0)
- added D102: 1N4148, Diode_SMD:D_MiniMELF, B.Cu at (118.8, 101.5)
- added D103: 1N4148, Diode_SMD:D_MiniMELF, B.Cu at (118.8, 98.5)
- added D104: 1N4148, Diode_SMD:D_MiniMELF, B.Cu at (123.2, 109.0)
- added D105: 1N4148, Diode_SMD:D_MiniMELF, B.Cu at (127.0, 142.5)
- added D106: 1N4148, Diode_SMD:D_MiniMELF, B.Cu at (127.0, 132.5)
- added D107: 1N4148, Diode_SMD:D_MiniMELF, B.Cu at (126.8, 122.5)
- added D108: 1N4148, Diode_SMD:D_MiniMELF, B.Cu at (126.8, 119.5)
- added D109: On LED, AJ:D_0805_AJ, F.Cu at (132.0, 51.5)
- added D110: 1N4007, Diode_SMD:D_MiniMELF, F.Cu at (132.2, 65.0)
- added D111: 1N4007, Diode_SMD:D_MiniMELF, F.Cu at (124.8, 65.0)
- added D201: On LED +, AJ:D_0805_AJ, F.Cu at (53.0, 90.0)
- added D202: On LED -, AJ:D_0805_AJ, F.Cu at (53.0, 100.0)
- added D203: 1N4007, Diode_SMD:D_MiniMELF, F.Cu at (76.0, 79.2)
- added D204: 1N4007, Diode_SMD:D_MiniMELF, F.Cu at (76.0, 123.5)
- added D401: +12V, AJ:D_0805_AJ, F.Cu at (110.0, 65.8)
- added D402: +5V, AJ:D_0805_AJ, F.Cu at (110.0, 78.8)
- added D403: -12v, AJ:D_0805_AJ, F.Cu at (110.0, 105.0)
- added D404: 1N4007, Diode_SMD:D_MiniMELF, B.Cu at (107.8, 139.2)
- added D405: 1N4007, Diode_SMD:D_MiniMELF, B.Cu at (107.5, 116.0)
- added G***: LOGO, AJ:Johansen_engineering_logo_20mm, F.Cu at (95.0, 127.5)
- added G***: LOGO, AJ:Johansen_engineering_logo_20mm, F.Cu at (141.8, 117.8)
- added G***: LOGO, AJ:Johansen_engineering_soldermask_20mm, F.Cu at (58.5, 52.2)
- added G***: LOGO, AJ:Johansen_engineering_soldermask_20mm, F.Cu at (87.5, 95.0)
- added G***: LOGO, AJ:Johansen_engineering_logo_20mm, F.Cu at (81.0, 52.2)
- added H103: MountingHole_Pad, AJ:MountingHole_Eurorack3, B.Cu at (107.5, 53.0)
- added H103: MountingHole_Pad, AJ:MountingHole_Eurorack3, B.Cu at (96.5, 53.0)
- added H103: MountingHole_Pad, AJ:MountingHole_Eurorack3, B.Cu at (107.5, 147.2)
- added H103: MountingHole_Pad, AJ:MountingHole_Eurorack3, B.Cu at (96.5, 147.2)
- added J101: Snare, Connector_Audio:Jack_3.5mm_QingPu_WQP-PJ398SM_Vertical_CircularHoles, F.Cu at (128.5, 105.0)
- added J102: LCymbals, Connector_Audio:Jack_3.5mm_QingPu_WQP-PJ398SM_Vertical_CircularHoles, F.Cu at (128.5, 85.0)
- added J103: SCymbals, Connector_Audio:Jack_3.5mm_QingPu_WQP-PJ398SM_Vertical_CircularHoles, F.Cu at (128.5, 75.0)
- added J104: Maracas, Connector_Audio:Jack_3.5mm_QingPu_WQP-PJ398SM_Vertical_CircularHoles, F.Cu at (128.5, 95.0)
- added J105: Bass, Connector_Audio:Jack_3.5mm_QingPu_WQP-PJ398SM_Vertical_CircularHoles, F.Cu at (128.6, 145.0)
- added J106: LBongo, Connector_Audio:Jack_3.5mm_QingPu_WQP-PJ398SM_Vertical_CircularHoles, F.Cu at (128.5, 135.0)
- added J107: HBongo, Connector_Audio:Jack_3.5mm_QingPu_WQP-PJ398SM_Vertical_CircularHoles, F.Cu at (128.5, 125.0)
- added J108: Claves, Connector_Audio:Jack_3.5mm_QingPu_WQP-PJ398SM_Vertical_CircularHoles, F.Cu at (128.5, 115.0)
- added J201: AudioJack2_SwitchT, Connector_Audio:Jack_3.5mm_Switronic_ST-005-G_horizontal, F.Cu at (75.0, 142.0)
- added J202: AudioJack2_SwitchT, Connector_Audio:Jack_3.5mm_Switronic_ST-005-G_horizontal, F.Cu at (65.0, 142.0)
- added J203: AudioJack2_SwitchT, Connector_Audio:Jack_3.5mm_Switronic_ST-005-G_horizontal, F.Cu at (55.0, 142.0)
- added J204: Power +, Connector_PinHeader_2.54mm:PinHeader_2x02_P2.54mm_Vertical, F.Cu at (86.5, 78.0)
- added J205: Power -, Connector_PinHeader_2.54mm:PinHeader_2x02_P2.54mm_Vertical, F.Cu at (86.5, 122.5)
- added J206: Conn_01x03_Male, Connector_PinHeader_2.54mm:PinHeader_1x03_P2.54mm_Vertical, F.Cu at (87.5, 142.0)
- added J207: Conn_01x03_Male, Connector_PinHeader_2.54mm:PinHeader_1x03_P2.54mm_Vertical, F.Cu at (87.5, 131.5)
- added J208: Conn_01x03_Male, Connector_PinHeader_2.54mm:PinHeader_1x03_P2.54mm_Vertical, F.Cu at (57.5, 131.0)
- added J209: Conn_01x03_Male, Connector_PinHeader_2.54mm:PinHeader_1x03_P2.54mm_Vertical, F.Cu at (87.0, 67.0)
- added J210: Conn_01x02_Male, Connector_PinHeader_2.54mm:PinHeader_1x02_P2.54mm_Vertical, F.Cu at (87.5, 108.0)
- added J301: Tone/Noise, Connector_PinHeader_2.54mm:PinHeader_1x03_P2.54mm_Vertical, B.Cu at (140.0, 129.0)
- added J302: RND, Connector_Audio:Jack_3.5mm_QingPu_WQP-PJ398SM_Vertical_CircularHoles, F.Cu at (148.5, 135.0)
- added J303: Noise, Connector_Audio:Jack_3.5mm_QingPu_WQP-PJ398SM_Vertical_CircularHoles, F.Cu at (148.5, 125.0)
- added J304: DRUM_OUT, Connector_Audio:Jack_3.5mm_QingPu_WQP-PJ398SM_Vertical_CircularHoles, F.Cu at (148.5, 145.0)
- added J401: Tone/Noise, Connector_PinHeader_2.54mm:PinHeader_1x04_P2.54mm_Vertical_SMD_Pin1Left, B.Cu at (107.8, 127.2)
- added L103: 100mH, Inductor_SMD:L_1206_3216Metric, B.Cu at (143.5, 97.5)
- added L104: 100mH, Inductor_SMD:L_1206_3216Metric, B.Cu at (140.5, 97.5)
- added P101: HEADER_2x8_Doepfer, Connector_IDC:IDC-Header_2x08_P2.54mm_Vertical, B.Cu at (122.8, 55.0)
- added P201: HEADER_2x5_Doepfer, Connector_IDC:IDC-Header_2x05_P2.54mm_Vertical, F.Cu at (63.0, 100.0)
- added P401: HEADER_2x8_Doepfer, Connector_IDC:IDC-Header_2x08_P2.54mm_Vertical, F.Cu at (100.8, 119.5)
- added Q101: 2N3904, Package_TO_SOT_SMD:SOT-23_Handsoldering, B.Cu at (129.5, 108.5)
- added Q102: 2N3904, Package_TO_SOT_SMD:SOT-23_Handsoldering, B.Cu at (142.0, 122.0)
- added Q103: 2N3904, Package_TO_SOT_SMD:SOT-23_Handsoldering, B.Cu at (142.0, 116.5)
- added Q104: 2N3904, Package_TO_SOT_SMD:SOT-23_Handsoldering, B.Cu at (133.0, 93.0)
- added R101: 10k, AJ:R_0805_AJ, B.Cu at (127.0, 82.0)
- added R102: 22k, AJ:R_0805_AJ, B.Cu at (120.0, 92.0)
- added R103: 10k, AJ:R_0805_AJ, B.Cu at (117.0, 79.0)
- added R104: 12k, AJ:R_0805_AJ, B.Cu at (121.0, 147.0)
- added R105: 12k, AJ:R_0805_AJ, B.Cu at (121.0, 137.5)
- added R106: 22k, AJ:R_0805_AJ, B.Cu at (121.0, 107.0)
- added R107: 47k, AJ:R_0805_AJ, B.Cu at (121.0, 149.0)
- added R108: 47k, AJ:R_0805_AJ, B.Cu at (121.0, 139.5)
- added R109: 1M, AJ:R_0805_AJ, B.Cu at (123.0, 81.5)
- added R110: 1M, AJ:R_0805_AJ, B.Cu at (123.0, 77.5)
- added R111: 27k, AJ:R_0805_AJ, B.Cu at (121.0, 142.5)
- added R112: 27k, AJ:R_0805_AJ, B.Cu at (121.0, 132.5)
- added R113: 100k, AJ:R_0805_AJ, B.Cu at (123.5, 98.5)
- added R114: 2k2, AJ:R_0805_AJ, B.Cu at (121.0, 113.0)
- added R115: 470k, AJ:R_0805_AJ, B.Cu at (127.5, 98.5)
- added R116: 10k, AJ:R_0805_AJ, B.Cu at (131.5, 142.5)
- added R117: 10k, AJ:R_0805_AJ, B.Cu at (131.5, 132.5)
- added R118: 1M, AJ:R_0805_AJ, B.Cu at (121.0, 111.0)
- added R119: 150k, AJ:R_0805_AJ, B.Cu at (146.0, 63.5)
- added R120: 68k, AJ:R_0805_AJ, B.Cu at (144.0, 63.5)
- added R121: 150k, AJ:R_0805_AJ, B.Cu at (146.0, 79.5)
- added R122: 68k, AJ:R_0805_AJ, B.Cu at (144.0, 79.5)
- added R123: 1M, AJ:R_0805_AJ, B.Cu at (128.5, 93.0)
- added R124: 0-470k, AJ:R_0805_AJ, B.Cu at (146.0, 67.5)
- added R125: 68k, AJ:R_0805_AJ, B.Cu at (144.0, 67.5)
- added R126: 0-470k, AJ:R_0805_AJ, B.Cu at (146.0, 83.5)
- added R127: 68k, AJ:R_0805_AJ, B.Cu at (144.0, 83.4)
- added R128: 1M, AJ:R_0805_AJ, B.Cu at (137.0, 116.5)
- added R129: 4k7, AJ:R_0805_AJ, B.Cu at (147.0, 97.5)
- added R130: 4k7, AJ:R_0805_AJ, B.Cu at (137.5, 97.5)
- added R131: 22k, AJ:R_0805_AJ, B.Cu at (142.0, 109.0)
- added R132: 12k, AJ:R_0805_AJ, B.Cu at (121.0, 127.5)
- added R133: 12k, AJ:R_0805_AJ, B.Cu at (121.0, 117.5)
- added R134: 47k, AJ:R_0805_AJ, B.Cu at (121.0, 129.5)
- added R135: 47k, AJ:R_0805_AJ, B.Cu at (121.0, 119.5)
- added R136: 27k, AJ:R_0805_AJ, B.Cu at (121.0, 121.5)
- added R137: 27k, AJ:R_0805_AJ, B.Cu at (121.0, 125.5)
- added R138: 22k, AJ:R_0805_AJ, F.Cu at (136.5, 51.5)
- added R139: 10k, AJ:R_0805_AJ, B.Cu at (131.5, 122.5)
- added R140: 10k, AJ:R_0805_AJ, B.Cu at (131.5, 119.5)
- added R141: 150k, AJ:R_0805_AJ, B.Cu at (146.0, 71.5)
- added R142: 68k, AJ:R_0805_AJ, B.Cu at (144.0, 71.5)
- added R143: 150k, AJ:R_0805_AJ, B.Cu at (133.5, 83.5)
- added R144: 68k, AJ:R_0805_AJ, B.Cu at (135.5, 83.5)
- added R145: 10R, AJ:R_0805_AJ, F.Cu at (124.0, 60.0)
- added R146: 10R, AJ:R_0805_AJ, F.Cu at (136.5, 60.0)
- added R147: 0-470k, AJ:R_0805_AJ, B.Cu at (146.0, 75.5)
- added R148: 68k, AJ:R_0805_AJ, B.Cu at (144.0, 75.5)
- added R149: 0-470k, AJ:R_0805_AJ, B.Cu at (133.5, 79.5)
- added R150: 68k, AJ:R_0805_AJ, B.Cu at (135.5, 79.5)
- added R151: 10R, AJ:R_0805_AJ, F.Cu at (131.5, 60.0)
- added R201: 22k, AJ:R_0805_AJ, F.Cu at (53.0, 86.0)
- added R202: 22k, AJ:R_0805_AJ, F.Cu at (53.0, 104.0)
- added R203: 10R, AJ:R_0805_AJ, F.Cu at (69.0, 86.0)
- added R204: 10R, AJ:R_0805_AJ, F.Cu at (69.0, 104.0)
- added R205: OPEN, AJ:R_0805_AJ, F.Cu at (79.5, 67.5)
- added R206: OPEN, AJ:R_0805_AJ, F.Cu at (79.5, 71.5)
- added R301: 100k, AJ:R_0805_AJ, B.Cu at (125.0, 66.0)
- added R302: 100k, AJ:R_0805_AJ, B.Cu at (125.0, 70.0)
- added R303: 470k, AJ:R_0805_AJ, F.Cu at (138.0, 79.0)
- added R304: 390k, AJ:R_0805_AJ, F.Cu at (140.0, 79.0)
- added R305: 390k, AJ:R_0805_AJ, F.Cu at (142.0, 79.0)
- added R306: 390k, AJ:R_0805_AJ, F.Cu at (144.0, 79.0)
- added R307: 100k, AJ:R_0805_AJ, B.Cu at (128.0, 69.0)
- added R308: 10k, AJ:R_0805_AJ, F.Cu at (145.5, 88.5)
- added R309: 10k, AJ:R_0805_AJ, F.Cu at (145.5, 92.5)
- added R310: OPEN, AJ:R_0805_AJ, F.Cu at (147.5, 88.5)
- added R311: 10k, AJ:R_0805_AJ, B.Cu at (137.0, 129.0)
- added R312: 0R, AJ:R_0805_AJ, F.Cu at (147.5, 92.5)
- added R313: 22k, AJ:R_0805_AJ, F.Cu at (132.5, 89.5)
- added R314: 1k, AJ:R_0805_AJ, F.Cu at (137.0, 86.0)
- added R315: 470r, AJ:R_0805_AJ, B.Cu at (137.0, 141.5)
- added R316: 22k, AJ:R_0805_AJ, F.Cu at (132.5, 91.5)
- added R323: 470R, AJ:R_0805_AJ, B.Cu at (137.0, 132.0)
- added R401: 0R, AJ:R_0805_AJ, B.Cu at (97.0, 134.2)
- added R402: 0R, AJ:R_0805_AJ, B.Cu at (97.0, 129.8)
- added R403: 0R, AJ:R_0805_AJ, B.Cu at (97.0, 119.5)
- added R404: 22k, AJ:R_0805_AJ, B.Cu at (110.0, 65.8)
- added R405: 10k, AJ:R_0805_AJ, B.Cu at (110.0, 78.8)
- added R406: 22k, AJ:R_0805_AJ, B.Cu at (110.0, 105.2)
- added R407: 10R, AJ:R_0805_AJ, B.Cu at (106.0, 135.5)
- added R408: 10R, AJ:R_0805_AJ, B.Cu at (109.5, 135.5)
- added R409: 10R, AJ:R_0805_AJ, B.Cu at (109.2, 119.7)
- added REF**: MountingHole_8.4mm_M8, MountingHole:MountingHole_8.4mm_M8, F.Cu at (101.8, 66.0)
- added REF**: MountingHole_8.4mm_M8, MountingHole:MountingHole_8.4mm_M8, F.Cu at (102.0, 79.0)
- added REF**: MountingHole_8.4mm_M8, MountingHole:MountingHole_8.4mm_M8, F.Cu at (102.0, 92.0)
- added REF**: MountingHole_8.4mm_M8, MountingHole:MountingHole_8.4mm_M8, F.Cu at (102.0, 105.0)
- added RV101: R_POT_TRIM, Potentiometer_THT:Potentiometer_Bourns_3296W_Vertical, B.Cu at (133.0, 98.5)
- added RV102: 220k, AJ:Potentiometer_China_RK09_Single_Vertical_AJ, F.Cu at (144.5, 112.5)
- added RV201: 100k, AJ:Potentiometer_China_RK09_Single_Vertical_AJ, F.Cu at (64.5, 72.5)
- added SW201: SW_SPDT, Button_Switch_THT:SW_PUSH_6mm_H8mm, F.Cu at (54.0, 113.0)
- added U101: 74HC04, Package_SO:SO-14_5.3x10.2mm_P1.27mm, B.Cu at (135.0, 70.0)
- added U302: TL072, AJ:AJ_SO-8_5.3x6.2mm_P1.27mm, F.Cu at (139.5, 90.0)
- moved TP105 60.0 mm to (223.0, 135.0)
- moved TP105 40.0 mm to (223.0, 125.0)
Routing:
- net +12Vc: track 0.00 -> 226.4 mm, vias 0 -> 4
- net +5V: track 0.00 -> 174.3 mm, vias 0 -> 4
- net GND: track 0.00 -> 173.4 mm, vias 0 -> 24
- net -12Vc: track 0.00 -> 128.2 mm, vias 0 -> 1
- net Net-(R323-Pad2): track 0.00 -> 106.0 mm
- net LBongoTrig: track 0.00 -> 102.2 mm, vias 0 -> 4
- net Net-(J301-Pad3): track 0.00 -> 97.2 mm, vias 0 -> 1
- net BassTrig: track 0.00 -> 93.2 mm
- net NoiseOut: track 0.00 -> 69.8 mm, vias 0 -> 7
- net HBongoTrig: track 0.00 -> 62.8 mm, vias 0 -> 6
- net Net-(R315-Pad2): track 0.00 -> 60.2 mm, vias 0 -> 5
- net Net-(J210-Pad1): track 0.00 -> 53.7 mm
- net Net-(J210-Pad2): track 0.00 -> 50.2 mm
- net ClavesTrig: track 0.00 -> 46.2 mm, vias 0 -> 6
- net Net-(J202-PadT): track 0.00 -> 32.3 mm
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- added copper zone on F.Cu, net (none)
Other:
- board size 40 x 128 mm -> 183 x 128 mm
- board text added: "BB-Power"
- board text added: "Drum78"
- board text added: "Drum78 - Rev A JE - 27/4-2021"
- board text added: "Hi"
- board text added: "KicadJE-BB-Power Johansen Engineering 22/4/2021 Rev A"
- board text added: "KicadJE-PDU1 27/4/2021 Rev A"
- board text added: "Long"
- board text added: "Low"
- board text added: "PDU1"
- board text added: "Shor"
- board text added: "Snr"
- board text added: "bass"
- board text added: "bongo"
- board text added: "claves"
- board text added: "cymbals"
- board text added: "maracas"
- board text added: "snare"
- board text removed: "Gain"
- board text removed: "HBg"
- board text removed: "LBg"
- board text removed: "LCym"
- board text removed: "SCym"
- board text removed: "Snare"
